Commit message: romeo moveit current progress

File: romeo_description/urdf/romeo.urdf (robot description, URDF)
Before this commit: robot romeo, 70 links, 69 joints
Joints:
- removed joint LFinger11
- removed joint RFinger11
- added joint LHand: type revolute, parent l_wrist, child LFinger11Link, origin xyz=0.10937 0.02468 0.00329 rpy=2.98023e-08 1.06465 0.122173, axis 0.121869 -0.992546 -4.37114e-08, limit lower=0 upper=1.06465082555556 effort=0 velocity=0
- added joint RHand: type revolute, parent r_wrist, child RFinger11Link, origin xyz=0.10937 -0.02468 0.00329 rpy=3.72529e-08 1.06465 -0.122173, axis -0.121869 -0.992546 -4.37114e-08, limit lower=0 upper=1.06465082555556 effort=0 velocity=0
- joint LFinger12: mimic joint=LFinger11 multiplier=1 offset=0 -> joint=LHand multiplier=1 offset=0
- joint LFinger13: mimic joint=LFinger11 multiplier=1 offset=0 -> joint=LHand multiplier=1 offset=0
- joint LFinger21: mimic joint=LFinger11 multiplier=1 offset=0 -> joint=LHand multiplier=1 offset=0
- joint LFinger22: mimic joint=LFinger11 multiplier=1 offset=0 -> joint=LHand multiplier=1 offset=0
- joint LFinger23: mimic joint=LFinger11 multiplier=1 offset=0 -> joint=LHand multiplier=1 offset=0
- joint LFinger31: mimic joint=LFinger11 multiplier=1 offset=0 -> joint=LHand multiplier=1 offset=0
- joint LFinger32: mimic joint=LFinger11 multiplier=1 offset=0 -> joint=LHand multiplier=1 offset=0
- joint LFinger33: mimic joint=LFinger11 multiplier=1 offset=0 -> joint=LHand multiplier=1 offset=0
- joint LThumb1: mimic joint=LFinger11 multiplier=-1 offset=0 -> joint=LHand multiplier=-1 offset=0
- joint LThumb2: mimic joint=LFinger11 multiplier=1 offset=0 -> joint=LHand multiplier=1 offset=0
- joint LThumb3: mimic joint=LFinger11 multiplier=1 offset=0 -> joint=LHand multiplier=1 offset=0
- joint RFinger12: mimic joint=RFinger11 multiplier=1 offset=0 -> joint=RHand multiplier=1 offset=0
- joint RFinger13: mimic joint=RFinger11 multiplier=1 offset=0 -> joint=RHand multiplier=1 offset=0
- joint RFinger21: mimic joint=RFinger11 multiplier=1 offset=0 -> joint=RHand multiplier=1 offset=0
- joint RFinger22: mimic joint=RFinger11 multiplier=1 offset=0 -> joint=RHand multiplier=1 offset=0
- joint RFinger23: mimic joint=RFinger11 multiplier=1 offset=0 -> joint=RHand multiplier=1 offset=0
- joint RFinger31: mimic joint=RFinger11 multiplier=1 offset=0 -> joint=RHand multiplier=1 offset=0
- joint RFinger32: mimic joint=RFinger11 multiplier=1 offset=0 -> joint=RHand multiplier=1 offset=0
- joint RFinger33: mimic joint=RFinger11 multiplier=1 offset=0 -> joint=RHand multiplier=1 offset=0
- joint RThumb1: mimic joint=RFinger11 multiplier=-1 offset=0 -> joint=RHand multiplier=-1 offset=0
- joint RThumb2: mimic joint=RFinger11 multiplier=1 offset=0 -> joint=RHand multiplier=1 offset=0
- joint RThumb3: mimic joint=RFinger11 multiplier=1 offset=0 -> joint=RHand multiplier=1 offset=0
